File: hardware/kicad/Untitled.kicad_pcb (KiCad board)
At the start: 2 copper layers, 22 x 30.5 mm, 7 parts, among them U1 TLC271IP

Commit message: schematics: fix tlc wireing
Connections:
- C2 pad 1: +3.3V -> GND
Routing:
- net GND: track 45.6 -> 53.9 mm
- net +3.3V: track 18.6 -> 13.6 mm
Changed lines of the file:
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@@
 			(layers "*.Cu" "*.Mask")
 			(remove_unused_layers no)
-			(net 3 "+3.3V")
+			(net 4 "GND")
 			(pintype "passive")
 		)
@@
 	(segment
 		(start 121.5272 75.03)
-		(end 122.4289 75.03)
+		(end 128.811 71.1752)
 		(width 0.2)
 		(layer "B.Cu")
-		(net 3)
-	)
-	(segment
-		(start 126.5272 75.03)
-		(end 122.4289 75.03)
-		(width 0.2)
-		(layer "B.Cu")
-		(net 3)
-	)
-	(segment
+		(net 4)
+	)
+	(segment
