File: hardware/kicad/Untitled.kicad_sch (KiCad schematic)
At the start: 7 parts, among them U1 TLC271IP

Commit message: schematics: fix tlc wireing
Connections:
- net +3.3V: no longer C2.1
- net GND: now also C2.1
Other:
- moved on the sheet: C2
